File: RGB LED/RGB LED.kicad_pcb (KiCad board)
At the start: 2 copper layers, 93.1 x 66.5 mm, 86 parts, among them J1 USB_C_Receptacle_USB2.0_16P, SW1 SW_SPST_FSMSM, SW2 SW_SPST_FSMSM, U1 AP2112K-3.3, U2 MAX7219, U3 ESP32-S3-WROOM-1-N4

Commit message: added name
Other:
- board text added: "Board by: Jeewoo Kang"
Changed lines of the file:
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@@
     (effects (font (size 1 1) (thickness 0.1)) (justify left bottom))
+  )
+  (gr_text "Board by: Jeewoo Kang" (at 139 105) (layer "F.Cu")
+    (effects (font (size 1.5 1.25) (thickness 0.3) bold) (justify left bottom))
   )
   (gr_text "ESP32" (at 123.8234 67.4036) (layer "Cmts.User")
